Commit message: Visual overhaul, smooth 1080p recorder and new 18 m showcase
Live view:
- Gazebo world: brick-coloured wall segments with pillars, chequered floor,
  sun shadows, sky and a clean full-window GUI that frames the maze.
  (Image textures were dropped: they made walls invisible to the robot camera.)
- RViz config generated per maze: centred, rotated to match Gazebo, docks
  hidden; travelled-path trail published by the explorer. rviz_render_mode
  gpu_override measured ~20-30 % CPU vs ~100-150 % in software mode.
- env.sh restores the WSLg X socket link after a WSL restart; the launch path
  no longer imports OpenCV (its Qt plugin path crashed the Gazebo GUI).

Recording:
- media_recorder rewritten: 1920x1080, 30 fps of simulated time streamed to
  H.264, frame-hold to keep 1x timing, plus 8x and ending-clip versions.
- Oblique/top-down recording cameras; real_time_factor launch argument.
- The robot turns to face the exit sign before reporting EXIT_REACHED.

New showcase (18 m x 18 m, 12x12): exit reached and verified, 209.6 m in
795.5 s, 0 contacts, 0 failed goals. Docs, README and post draft updated.

Co-Authored-By: Claude Opus 5.5 <noreply@anthropic.com>

File: src/mazemind_description/urdf/mazemind.urdf.xacro (robot description, xacro)
@@ -38,7 +38,7 @@
     <inertia ixx="${m*(y*y+z*z)/12}" ixy="0" ixz="0" iyy="${m*(x*x+z*z)/12}" iyz="0" izz="${m*(x*x+y*y)/12}"/>
   </xacro:macro>
-  <material name="body"><color rgba="0.15 0.35 0.75 1"/></material>
+  <material name="body"><color rgba="1.0 0.42 0.05 1"/></material>
   <material name="dark"><color rgba="0.1 0.1 0.1 1"/></material>
-  <material name="sensor"><color rgba="0.9 0.5 0.1 1"/></material>
+  <material name="sensor"><color rgba="0.15 0.15 0.17 1"/></material>
   <!-- ============================================================ base -->
   <link name="base_footprint"/>
